Commit message: version 2.0.0  3D lidar

File: urdf/bcr_bot.xacro (robot description, xacro)
@@ -25,4 +25,14 @@
     <xacro:property name="two_d_lidar_min_range" value="0.55"/>
     <xacro:property name="two_d_lidar_max_range" value="16"/>
+    <xacro:property name="three_d_lidar_update_rate" value="10"/>
+    <xacro:property name="three_d_lidar_horizontal_samples" value="1800"/>
+    <xacro:property name="three_d_lidar_vertical_samples" value="16"/>
+    <xacro:property name="three_d_lidar_horizontal_min_angle" value="-180"/>
+    <xacro:property name="three_d_lidar_horizontal_max_angle" value="180"/>
+    <xacro:property name="three_d_lidar_vertical_min_angle" value="-15"/>
+    <xacro:property name="three_d_lidar_vertical_max_angle" value="15"/>
+    <xacro:property name="three_d_lidar_min_range" value="0.3"/>
+    <xacro:property name="three_d_lidar_max_range" value="100"/>
+    <xacro:arg name="three_d_lidar_enabled" default="false" />
     <xacro:property name="camera_baseline" value="0.06"/>
     <xacro:property name="camera_height" value="0.10"/>
@@ -126,4 +136,26 @@
         </gazebo>
     </xacro:if>
+    <!-- ............................. 3D LIDAR ........................................ -->
+    <xacro:if value="$(arg three_d_lidar_enabled)">
+        <link name="three_d_lidar">
+            <visual>
+                <origin xyz="0 0 0" rpy="0 0 0" />
+                <geometry>
+                    <cylinder length="0.07" radius="0.05"/>
+                </geometry>
+                <material name="black"/>
+            </visual>
+            <inertial>
+                <origin xyz="0 0 0" rpy="0 0 0" />
+                <mass value="0.83"/>
+                <xacro:cylinder_inertia m="0.83" r="0.05" h="0.07"/>
+            </inertial>
+        </link>
+        <joint name="three_d_lidar_joint" type="fixed">
+            <parent link="base_link"/>
+            <child link="three_d_lidar"/>
+            <origin xyz="0.0 0 0.155" rpy="0 0 0" />
+        </joint>
+    </xacro:if>
     <!-- ............................. IMU ........................................ -->
     <link name="imu_frame"/>

File: urdf/gz.xacro (robot description, xacro)
@@ -72,4 +72,38 @@
         </gazebo>
     </xacro:if>
+    <!-- ........................... 3D LIDAR config ................................... -->
+    <xacro:if value="$(arg three_d_lidar_enabled)">
+        <gazebo reference="three_d_lidar">
+            <material>Gazebo/Black</material>
+            <sensor name='gpu_3d_lidar' type='gpu_lidar'>
+                <topic>three_d_lidar_points</topic>
+                <update_rate>${three_d_lidar_update_rate}</update_rate>
+                <gz_frame_id>three_d_lidar</gz_frame_id>
+                <lidar>
+                    <scan>
+                        <horizontal>
+                            <samples>${three_d_lidar_horizontal_samples}</samples>
+                            <resolution>1</resolution>
+                            <min_angle>${radians(three_d_lidar_horizontal_min_angle)}</min_angle>
+                            <max_angle>${radians(three_d_lidar_horizontal_max_angle)}</max_angle>
+                        </horizontal>
+                        <vertical>
+                            <samples>${three_d_lidar_vertical_samples}</samples>
+                            <resolution>1</resolution>
+                            <min_angle>${radians(three_d_lidar_vertical_min_angle)}</min_angle>
+                            <max_angle>${radians(three_d_lidar_vertical_max_angle)}</max_angle>
+                        </vertical>
+                    </scan>
+                    <range>
+                        <min>${three_d_lidar_min_range}</min>
+                        <max>${three_d_lidar_max_range}</max>
+                        <resolution>0.01</resolution>
+                    </range>
+                </lidar>
+                <always_on>1</always_on>
+                <visualize>true</visualize>
+            </sensor>
+        </gazebo>
+    </xacro:if>
     <!-- ........................... CAMERA config ................................... -->
     <xacro:if value="$(arg camera_enabled)">
@@ -89,5 +123,5 @@
                     <clip>
                         <near>0.05</near>
-                        <far>8.0</far>
+                        <far>20.0</far>
                     </clip>
                 </camera>

Commit message: version 2.0.1

File: urdf/bcr_bot.xacro (robot description, xacro)
@@ -26,8 +26,8 @@
     <xacro:property name="two_d_lidar_max_range" value="16"/>
     <xacro:property name="three_d_lidar_update_rate" value="10"/>
-    <xacro:property name="three_d_lidar_horizontal_samples" value="1800"/>
+    <xacro:property name="three_d_lidar_horizontal_samples" value="600"/>
     <xacro:property name="three_d_lidar_vertical_samples" value="16"/>
-    <xacro:property name="three_d_lidar_horizontal_min_angle" value="-180"/>
-    <xacro:property name="three_d_lidar_horizontal_max_angle" value="180"/>
+    <xacro:property name="three_d_lidar_horizontal_min_angle" value="-60"/>
+    <xacro:property name="three_d_lidar_horizontal_max_angle" value="60"/>
     <xacro:property name="three_d_lidar_vertical_min_angle" value="-15"/>
     <xacro:property name="three_d_lidar_vertical_max_angle" value="15"/>

Commit message: version 2.0.1.3

File: urdf/bcr_bot.xacro (robot description, xacro)
@@ -30,6 +30,6 @@
     <xacro:property name="three_d_lidar_horizontal_min_angle" value="-60"/>
     <xacro:property name="three_d_lidar_horizontal_max_angle" value="60"/>
-    <xacro:property name="three_d_lidar_vertical_min_angle" value="-15"/>
-    <xacro:property name="three_d_lidar_vertical_max_angle" value="15"/>
+    <xacro:property name="three_d_lidar_vertical_min_angle" value="-20"/>
+    <xacro:property name="three_d_lidar_vertical_max_angle" value="10"/>
     <xacro:property name="three_d_lidar_min_range" value="0.3"/>
     <xacro:property name="three_d_lidar_max_range" value="100"/>
@@ -155,5 +155,5 @@
             <parent link="base_link"/>
             <child link="three_d_lidar"/>
-            <origin xyz="0.0 0 0.155" rpy="0 0 0" />
+            <origin xyz="${chassis_length/2} 0 0.155" rpy="0 0 0" />
         </joint>
     </xacro:if>
