Commit message: temp

File: robot/urdf/bcr_bot.xacro (robot description, xacro)
@@ -53,17 +53,17 @@
     <xacro:property name="odometry_source" value="$(arg odometry_source)"/>
     <!-- ............................... LOAD MACROS ................................. -->
-    <xacro:include filename="$(find bcr_bot)/urdf/materials.xacro"/>
-    <xacro:include filename="$(find bcr_bot)/urdf/macros.xacro"/>
+    <xacro:include filename="$(find bcr_bot)/robot/urdf/materials.xacro"/>
+    <xacro:include filename="$(find bcr_bot)/robot/urdf/macros.xacro"/>
     <xacro:if value="$(arg sim_gazebo)">
-        <xacro:include filename="$(find bcr_bot)/urdf/gazebo.xacro"/>
+        <xacro:include filename="$(find bcr_bot)/robot/urdf/gazebo.xacro"/>
     </xacro:if>
     <xacro:if value="$(arg sim_ign)">
-        <xacro:include filename="$(find bcr_bot)/urdf/ign.xacro"/>
+        <xacro:include filename="$(find bcr_bot)/robot/urdf/ign.xacro"/>
     </xacro:if>
     <xacro:if value="$(arg sim_gz)">
-        <xacro:include filename="$(find bcr_bot)/urdf/gz.xacro"/>
+        <xacro:include filename="$(find bcr_bot)/robot/urdf/gz.xacro"/>
     </xacro:if>
     <xacro:if value="$(arg sim_mujoco)">
-        <xacro:include filename="$(find bcr_bot)/urdf/mujoco_ros2_control.xacro"/>
+        <xacro:include filename="$(find bcr_bot)/robot/urdf/mujoco_ros2_control.xacro"/>
     </xacro:if>
     <!-- ................................ BASE LINK .................................. -->
@@ -85,5 +85,5 @@
             <origin xyz="0 0 -0.205" rpy="0 0 0" />
             <geometry>
-                <mesh filename="file://$(find bcr_bot)/meshes/bcr_bot_mesh.dae" scale="1 1 1"/>
+                <mesh filename="file://$(find bcr_bot)/robot/meshes/bcr_bot_mesh.dae" scale="1 1 1"/>
             </geometry>
         </visual>
@@ -178,5 +178,5 @@
                 <origin xyz="0 0 0" rpy="0 0 0" />
                 <geometry>
-                    <mesh filename="file://$(find bcr_bot)/meshes/kinect/d415.dae"/>
+                    <mesh filename="file://$(find bcr_bot)/robot/meshes/kinect/d415.dae"/>
                 </geometry>
                 <material name="black"/>
@@ -212,5 +212,5 @@
                 <origin xyz="0 0 0" rpy="0 0 0" />
                 <geometry>
-                    <mesh filename="file://$(find bcr_bot)/meshes/kinect/d415.dae"/>
+                    <mesh filename="file://$(find bcr_bot)/robot/meshes/kinect/d415.dae"/>
                 </geometry>
                 <material name="black"/>
